Commit message: doesn't work

File: robotiq_85_gripper/robotiq_85_description/urdf/robotiq_85_gripper.urdf.xacro (robot description, xacro)
@@ -2,10 +2,10 @@
 <robot name="robotiq_85_gripper" xmlns:xacro="http://ros.org/wiki/xacro">
     <xacro:include filename="$(find robotiq_85_description)/urdf/robotiq_85_gripper.transmission.xacro" />
-    <xacro:macro name="robotiq_85_gripper" params="prefix parent *origin">
-        <joint name="${prefix}gripper_base_joint" type="fixed">
+    <xacro:macro name="robotiq_85_gripper" params="prefix">
+        <!-- <joint name="${prefix}gripper_base_joint" type="fixed">
             <parent link="${parent}"/>
             <child link="${prefix}gripper_base_link"/>
             <xacro:insert_block name="origin"/>
-        </joint>
+        </joint> -->
         <link name="${prefix}gripper_base_link">
             <visual>
@@ -303,5 +303,5 @@
             <arm>
               <arm_name>gripper_arm</arm_name>
-              <palm_link>${parent}</palm_link>
+              <palm_link>${prefix}gripper_coupling_link</palm_link>
               <gripper_link>${prefix}gripper_finger1_finger_tip_link</gripper_link>
               <gripper_link>${prefix}gripper_finger2_finger_tip_link</gripper_link>

File: vention_conveyor/vention_conveyor_description/urdf/workbench.urdf.xacro (robot description, xacro)
@@ -4,34 +4,16 @@
      For more information, please see http://wiki.ros.org/sw_urdf_exporter -->
 <robot xmlns:xacro="http://ros.org/wiki/xacro" name="workbench">
-    <xacro:macro name="workbench" params="parent prefix *origin">
+    <xacro:macro name="workbench" params="prefix">
         <!-- mount the workbench to the robot -->
-        <joint name="${prefix}workbench_fix" type="fixed">
-        <xacro:insert_block name="origin" />
-        <parent link="${parent}" />
-        <child link="${prefix}workbench_table" />
-        </joint>
         <link
-            name="workbench_table">
-            <inertial>
-            <origin
-                xyz="0.42892 0.020265 -0.31198"
-                rpy="0 0 0" />
-            <mass
-                value="53.725" />
-            <inertia
-                ixx="2.969"
-                ixy="1.6142E-06"
-                ixz="-0.00010958"
-                iyy="1.6706"
-                iyz="-2.7677E-06"
-                izz="3.987" />
-            </inertial>
+            name="${prefix}workbench_link">
             <visual>
             <origin
-                xyz="0 0 0"
+                xyz="-0.25 -.943 -1.01"
                 rpy="0 0 0" />
             <geometry>
                 <mesh
-                filename="package://vention_conveyor_description/meshes/workbench_table.STL" />
+                filename="package://workbench/meshes/workbench_base.STL" />
+                <!-- <box size="2 2 1"/> -->
             </geometry>
             <material
@@ -43,18 +25,46 @@
             <collision>
             <origin
-                xyz="0 0 0"
+                xyz="-0.25 -.943 -1.01"
                 rpy="0 0 0" />
             <geometry>
                 <mesh
-                filename="package://vention_conveyor_description/meshes/workbench_table.STL" />
+                filename="package://workbench/meshes/workbench_base.STL" />
             </geometry>
             </collision>
         </link>
-        <joint name="${prefix}mounting_joint" type="fixed">
-        <origin xyz="0 0 0" rpy="0 0 0" />
-        <parent link="${prefix}workbench_table" />
-        <child link="${prefix}mounting_link" />
+        <joint name="${prefix}axis1_joint" type="prismatic">
+            <parent link="${prefix}workbench_link"/>
+            <child link="${prefix}axis1"/>
+            <!-- Here we enter the joint position just defined before -->
+            <origin xyz="0 0 0" rpy="0 0 0"/>
+            <!-- Here we define the axis along which the geometry is moved -->
+            <axis xyz="0 1 0"/>
+            <!-- Here we define the joint's upper and lower limits -->
+            <limit effort="1000.0" lower="-.5" upper=".5" velocity="0.05"/>
         </joint>
-        <link name="${prefix}mounting_link"/>
+        <link name="${prefix}axis1">
+            <visual>
+                <geometry>
+                    <mesh
+                    filename="package://workbench/meshes/workbench_mount.STL" />
+                </geometry>
+                <origin
+                xyz="-.09 -.09 0"
+                rpy="0 0 0" />
+                <material name="">
+                    <color
+                    rgba="0.33725 0.52941 0.75686 1" />
+                </material>
+            </visual>
+            <collision>
+                <geometry>
+                    <mesh
+                    filename="package://workbench/meshes/workbench_mount.STL" />
+                </geometry>
+                <origin
+                xyz="-.09 -.09 0"
+                rpy="0 0 0" />
+            </collision>
+        </link>
     </xacro:macro>
 </robot>

Commit message: everything working confirmed, including azure kinect

File: robotiq_85_gripper/robotiq_85_description/urdf/robotiq_85_gripper.urdf.xacro (robot description, xacro)
@@ -2,10 +2,10 @@
 <robot name="robotiq_85_gripper" xmlns:xacro="http://ros.org/wiki/xacro">
     <xacro:include filename="$(find robotiq_85_description)/urdf/robotiq_85_gripper.transmission.xacro" />
-    <xacro:macro name="robotiq_85_gripper" params="prefix">
-        <!-- <joint name="${prefix}gripper_base_joint" type="fixed">
+    <xacro:macro name="robotiq_85_gripper" params="prefix parent *origin">
+        <joint name="${prefix}gripper_base_joint" type="fixed">
             <parent link="${parent}"/>
             <child link="${prefix}gripper_base_link"/>
             <xacro:insert_block name="origin"/>
-        </joint> -->
+        </joint>
         <link name="${prefix}gripper_base_link">
             <visual>
@@ -303,5 +303,5 @@
             <arm>
               <arm_name>gripper_arm</arm_name>
-              <palm_link>${prefix}gripper_coupling_link</palm_link>
+              <palm_link>${parent}</palm_link>
               <gripper_link>${prefix}gripper_finger1_finger_tip_link</gripper_link>
               <gripper_link>${prefix}gripper_finger2_finger_tip_link</gripper_link>
