Commit message: created launch file in pycontrol package

File: Azure_Kinect_ROS_Driver/urdf/camera_mount.urdf.xacro (robot description, xacro)
@@ -38,4 +38,6 @@
             <origin xyz="0 0 0" rpy="0. 0. 0." />
         </joint>
+        <link name="${prefix}tool_link"/>
+        <link name="${prefix}camera_link"/>
     </xacro:macro>
 </robot>

File: pycontrol/urdf/ur5e_workbench.urdf.xacro (robot description, xacro)
@@ -42,4 +42,9 @@
         <origin xyz="0.05 0.0375 0.04" rpy="${pi/2} ${pi} 0"/>
     </xacro:azure_camera_mount>
+    <!-- ############### CAMERA ################ -->
+    <xacro:include filename="$(find azure_kinect_ros_driver)/urdf/azure_kinect.urdf.xacro" />
+    <xacro:azure_kinect prefix="${prefix}" parent="${prefix}camera_link" >
+        <origin xyz="0.05 -0.04 0.106" rpy="0 0 ${-pi/2}"/>
+    </xacro:azure_kinect>
     <!-- ############### GRIPPER ################ -->
     <xacro:include filename="$(find robotiq_85_description)/urdf/robotiq_85_gripper.urdf.xacro" />
@@ -54,4 +59,7 @@
                 <cylinder radius="0.04" length="0.017"/>
             </geometry>
+            <material name="black">
+                <color rgba="1 1 1 1.0"/>
+            </material>
         </visual>
         <collision>
@@ -64,8 +72,3 @@
         <origin xyz="0 0 -0.008" rpy="0 ${pi/2} ${-pi/2}" />
     </xacro:robotiq_85_gripper>
-    <!-- ############### CAMERA ################ -->
-    <xacro:include filename="$(find azure_kinect_ros_driver)/urdf/azure_kinect.urdf.xacro" />
-    <xacro:azure_kinect prefix="${prefix}" parent="${prefix}camera_link" >
-        <origin xyz="0.05 -0.04 0.106" rpy="0 0 ${-pi/2}"/>
-    </xacro:azure_kinect>
 </robot>
